File: KiCad/Rx/Rx_Schematic/Rx_Schematic_V1_0/Rx_Schematic_V1_0.kicad_sch (KiCad schematic)
At the start: 2 parts, among them J1 Analog, J2 Digital

Commit message: Added data sheets and symbol for motor driver
Parts:
- added IC?: TB9051FTG, TB9051FTG, symbol TB9051FTG:TB9051FTG
- added U?: AMS1117-3.3, Package_TO_SOT_SMD:SOT-223-3_TabPin2, symbol Regulator_Linear:AMS1117-3.3
- added U?: NRF24L01_Breakout, RF_Module:nRF24L01_Breakout, symbol RF:NRF24L01_Breakout
Changed lines of the file:
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@@
     (pin "9")
+  )
+  (symbol (lib_id "Regulator_Linear:AMS1117-3.3") (at 128.27 26.67 0) (unit 1)
+    (in_bom yes) (on_board yes) (fields_autoplaced)
+    (property "Reference" "U?" (id 0) (at 128.27 19.05 0))
+    (property "Value" "AMS1117-3.3" (id 1) (at 128.27 21.59 0))
+    (property "Footprint" "Package_TO_SOT_SMD:SOT-223-3_TabPin2" (id 2) (at 128.27 21.59 0)
+      (effects (font (size 1.27 1.27)) hide)
+    )
+    (property "Datasheet" "http://www.advanced-monolithic.com/pdf/ds1117.pdf" (id 3) (at 130.81 33.02 0)
+      (effects (font (size 1.27 1.27)) hide)
+    )
+    (pin "1")
+    (pin "2")
+    (pin "3")
   )
   (symbol (lib_id "power:+5V") (at 26.67 24.13 0) (unit 1)
@@
     )
     (pin "1")
+  )
+  (symbol (lib_id "TB9051FTG:TB9051FTG") (at 73.66 127 0) (unit 1)
+    (in_bom yes) (on_board yes) (fields_autoplaced)
+    (property "Reference" "IC?" (id 0) (at 91.44 119.38 0))
+    (property "Value" "TB9051FTG" (id 1) (at 91.44 121.92 0))
+    (property "Footprint" "TB9051FTG" (id 2) (at 105.41 124.46 0)
+      (effects (font (size 1.27 1.27)) (justify left) hide)
+    )
+    (property "Datasheet" "https://toshiba.semicon-storage.com/ap-en/semiconductor/product/automotive-devices/detail.TB9051FTG.html" (id 3) (at 105.41 127 0)
+      (effects (font (size 1.27 1.27)) (justify left) hide)
+    )
+    (property "Description" "PWM type single channel H-Bridge DC brushed motor driver for automotive use" (id 4) (at 105.41 129.54 0)
+      (effects (font (size 1.27 1.27)) (justify left) hide)
+    )
+    (property "Height" "1.8" (id 5) (at 105.41 132.08 0)
+      (effects (font (size 1.27 1.27)) (justify left) hide)
+    )
+    (property "Manufacturer_Name" "Toshiba" (id 6) (at 105.41 134.62 0)
+      (effects (font (size 1.27 1.27)) (justify left) hide)
+    )
+    (property "Manufacturer_Part_Number" "TB9051FTG" (id 7) (at 105.41 137.16 0)
+      (effects (font (size 1.27 1.27)) (justify left) hide)
+    )
+    (property "Mouser Part Number" "" (id 8) (at 105.41 139.7 0)
+      (effects (font (size 1.27 1.27)) (justify left) hide)
+    )
+    (property "Mouser Price/Stock" "" (id 9) (at 105.41 142.24 0)
+      (effects (font (size 1.27 1.27)) (justify left) hide)
+    )
+    (property "Arrow Part Number" "" (id 10) (at 105.41 144.78 0)
+      (effects (font (size 1.27 1.27)) (justify left) hide)
+    )
+    (property "Arrow Price/Stock" "" (id 11) (at 105.41 147.32 0)
+      (effects (font (size 1.27 1.27)) (justify left) hide)
+    )
+    (pin "1")
+    (pin "10")
+    (pin "11")
+    (pin "12")
+    (pin "13")
+    (pin "14")
+    (pin "15")
+    (pin "16")
+    (pin "17")
+    (pin "18")
+    (pin "19")
+    (pin "2")
+    (pin "20")
+    (pin "21")
+    (pin "22")
+    (pin "23")
+    (pin "24")
+    (pin "25")
+    (pin "26")
+    (pin "27")
+    (pin "28")
+    (pin "29")
+    (pin "3")
+    (pin "4")
+    (pin "5")
+    (pin "6")
+    (pin "7")
+    (pin "8")
+    (pin "9")
+    (pin "C1")
+    (pin "C2")
+    (pin "C3")
+    (pin "C4")
+  )
+  (symbol (lib_id "RF:NRF24L01_Breakout") (at 149.86 48.26 0) (unit 1)
+    (in_bom yes) (on_board yes) (fields_autoplaced)
+    (property "Reference" "U?" (id 0) (at 160.02 46.9899 0)
+      (effects (font (size 1.27 1.27)) (justify left))
+    )
+    (property "Value" "NRF24L01_Breakout" (id 1) (at 160.02 49.5299 0)
+      (effects (font (size 1.27 1.27)) (justify left))
+    )
+    (property "Footprint" "RF_Module:nRF24L01_Breakout" (id 2) (at 153.67 33.02 0)
+      (effects (font (size 1.27 1.27) italic) (justify left) hide)
+    )
+    (property "Datasheet" "http://www.nordicsemi.com/eng/content/download/2730/34105/file/nRF24L01_Product_Specification_v2_0.pdf" (id 3) (at 149.86 50.8 0)
+      (effects (font (size 1.27 1.27)) hide)
+    )
+    (pin "1")
+    (pin "2")
+    (pin "3")
+    (pin "4")
+    (pin "5")
+    (pin "6")
+    (pin "7")
+    (pin "8")
   )
   (symbol (lib_id "power:GND") (at 29.21 72.39 0) (unit 1)
@@
       (reference "#PWR0105") (unit 1) (value "GND") (footprint "")
     )
+    (path "/c2551cd8-dcb5-4d44-943f-608f019fd027"
+      (reference "IC?") (unit 1) (value "TB9051FTG") (footprint "TB9051FTG")
+    )
     (path "/00000000-0000-0000-0000-000056d719df"
       (reference "J1") (unit 1) (value "Analog") (footprint "Connector_PinHeader_2.54mm:PinHeader_1x17_P2.54mm_Vertical")
@@
       (reference "J2") (unit 1) (value "Digital") (footprint "Connector_PinHeader_2.54mm:PinHeader_1x17_P2.54mm_Vertical")
     )
-  )
+    (path "/10d11b55-e7ba-4181-9a27-0ad11636ee7e"
+      (reference "U?") (unit 1) (value "AMS1117-3.3") (footprint "Package_TO_SOT_SMD:SOT-223-3_TabPin2")
+    )
+    (path "/cc42cce8-f999-466f-a2c1-976549ab2c86"
+      (reference "U?") (unit 1) (value "NRF24L01_Breakout") (footprint "RF_Module:nRF24L01_Breakout")
+    )
+  )
