File: KiCad/Rx/Rx_Schematic/Rx_Schematic_V1_0/Rx_Project/Rx_Project.kicad_sch (KiCad schematic)
At the start: 5 parts, among them J1 Conn_01x05, J2 Conn_01x02, J3 Conn_01x06, J4 Conn_01x02, U1 ProMicro

Commit message: Schematic finished
Connections:
- net at U1.13 (B6): now also J3.3 (Pin_3)
- net at U1.17 (F7): now also J1.4 (Pin_4)
- net at U1.18 (F6): now also J1.5 (Pin_5)
- net at U1.19 (F5): now also J2.1 (Pin_1)
- net at U1.20 (F4): now also J3.2 (Pin_2)
- net at U1.23 (GND): now also J2.2 (Pin_2)
- net at U1.3 (GND): now also J4.2 (Pin_2)
- net at U1.4 (GND): now also J3.1 (Pin_1)
- net at U1.8 (C6): now also J3.4 (Pin_4)
- net at U1.9 (D7): now also J3.5 (Pin_5)
Other:
- note added: "Motor Driver Connector"
- note added: "NRF Connector"
- note added: "NRF Power"
- moved on the sheet: J3
Changed lines of the file:
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@@
 (kicad_sch (version 20230121) (generator eeschema)
   (paper "A4")
+  (wire (pts (xy 57.15 81.28) (xy 52.07 81.28))
+    (stroke (width 0) (type default) (color 72 0 72 1))
+  )
   (wire (pts (xy 106.68 85.09) (xy 92.71 85.09))
     (stroke (width 0) (type default))
   )
+  (wire (pts (xy 104.14 116.84) (xy 129.54 116.84))
+    (stroke (width 0) (type default) (color 255 153 0 1))
+  )
   (wire (pts (xy 111.76 86.36) (xy 106.68 86.36))
     (stroke (width 0) (type default))
@@
     (stroke (width 0) (type default))
   )
+  (wire (pts (xy 129.54 66.04) (xy 129.54 60.96))
+    (stroke (width 0) (type default) (color 0 0 0 1))
+  )
   (wire (pts (xy 102.87 88.9) (xy 102.87 83.82))
-    (stroke (width 0) (type default))
+    (stroke (width 0) (type default) (color 0 0 255 1))
   )
   (wire (pts (xy 92.71 86.36) (xy 101.6 86.36))
-    (stroke (width 0) (type default))
+    (stroke (width 0) (type default) (color 128 77 0 1))
+  )
+  (wire (pts (xy 104.14 73.66) (xy 104.14 116.84))
+    (stroke (width 0) (type default) (color 255 153 0 1))
   )
   (wire (pts (xy 101.6 81.28) (xy 111.76 81.28))
-    (stroke (width 0) (type default))
+    (stroke (width 0) (type default) (color 128 77 0 1))
+  )
+  (wire (pts (xy 50.8 101.6) (xy 129.54 101.6))
+    (stroke (width 0) (type default) (color 0 0 0 1))
+  )
+  (wire (pts (xy 96.52 91.44) (xy 96.52 119.38))
+    (stroke (width 0) (type default) (color 128 77 0 1))
   )
   (wire (pts (xy 92.71 88.9) (xy 102.87 88.9))
-    (stroke (width 0) (type default))
+    (stroke (width 0) (type default) (color 0 0 255 1))
+  )
+  (wire (pts (xy 96.52 119.38) (xy 129.54 119.38))
+    (stroke (width 0) (type default) (color 128 77 0 1))
+  )
+  (wire (pts (xy 92.71 91.44) (xy 96.52 91.44))
+    (stroke (width 0) (type default) (color 128 77 0 1))
+  )
+  (wire (pts (xy 97.79 78.74) (xy 92.71 78.74))
+    (stroke (width 0) (type default) (color 255 153 0 1))
+  )
+  (wire (pts (xy 52.07 81.28) (xy 52.07 121.92))
+    (stroke (width 0) (type default) (color 72 0 72 1))
+  )
+  (wire (pts (xy 127 76.2) (xy 127 58.42))
+    (stroke (width 0) (type default) (color 255 0 0 1))
   )
   (wire (pts (xy 101.6 86.36) (xy 101.6 81.28))
-    (stroke (width 0) (type default))
+    (stroke (width 0) (type default) (color 128 77 0 1))
+  )
+  (wire (pts (xy 52.07 121.92) (xy 129.54 121.92))
+    (stroke (width 0) (type default) (color 72 0 72 1))
   )
   (wire (pts (xy 92.71 85.09) (xy 92.71 83.82))
     (stroke (width 0) (type default))
   )
+  (wire (pts (xy 111.76 91.44) (xy 97.79 91.44))
+    (stroke (width 0) (type default) (color 255 153 0 1))
+  )
+  (wire (pts (xy 53.34 124.46) (xy 129.54 124.46))
+    (stroke (width 0) (type default))
+  )
+  (wire (pts (xy 50.8 68.58) (xy 50.8 101.6))
+    (stroke (width 0) (type default) (color 0 0 0 1))
+  )
+  (wire (pts (xy 49.53 71.12) (xy 49.53 114.3))
+    (stroke (width 0) (type default) (color 0 0 0 1))
+  )
+  (wire (pts (xy 127 58.42) (xy 129.54 58.42))
+    (stroke (width 0) (type default) (color 255 0 0 1))
+  )
+  (wire (pts (xy 92.71 76.2) (xy 127 76.2))
+    (stroke (width 0) (type default) (color 255 0 0 1))
+  )
+  (wire (pts (xy 92.71 66.04) (xy 129.54 66.04))
+    (stroke (width 0) (type default) (color 0 0 0 1))
+  )
+  (wire (pts (xy 92.71 82.55) (xy 92.71 81.28))
+    (stroke (width 0) (type default) (color 255 255 0 1))
+  )
+  (wire (pts (xy 49.53 114.3) (xy 129.54 114.3))
+    (stroke (width 0) (type default) (color 0 0 0 1))
+  )
+  (wire (pts (xy 57.15 68.58) (xy 50.8 68.58))
+    (stroke (width 0) (type default) (color 0 0 0 1))
+  )
+  (wire (pts (xy 107.95 88.9) (xy 107.95 82.55))
+    (stroke (width 0) (type default) (color 255 255 0 1))
+  )
   (wire (pts (xy 102.87 83.82) (xy 111.76 83.82))
-    (stroke (width 0) (type default))
+    (stroke (width 0) (type default) (color 0 0 255 1))
+  )
+  (wire (pts (xy 97.79 91.44) (xy 97.79 78.74))
+    (stroke (width 0) (type default) (color 255 153 0 1))
+  )
+  (wire (pts (xy 57.15 71.12) (xy 49.53 71.12))
+    (stroke (width 0) (type default) (color 0 0 0 1))
+  )
+  (wire (pts (xy 53.34 83.82) (xy 53.34 124.46))
+    (stroke (width 0) (type default))
+  )
+  (wire (pts (xy 111.76 88.9) (xy 107.95 88.9))
+    (stroke (width 0) (type default) (color 255 255 0 1))
+  )
+  (wire (pts (xy 57.15 83.82) (xy 53.34 83.82))
+    (stroke (width 0) (type default))
+  )
+  (wire (pts (xy 92.71 73.66) (xy 104.14 73.66))
+    (stroke (width 0) (type default) (color 255 153 0 1))
+  )
+  (wire (pts (xy 107.95 82.55) (xy 92.71 82.55))
+    (stroke (width 0) (type default) (color 255 255 0 1))
+  )
+  (text "Motor Driver Connector\n" (at 135.89 125.73 0)
+    (effects (font (size 1.27 1.27)) (justify left bottom))
+  )
+  (text "NRF Connector\n" (at 116.84 90.17 0)
+    (effects (font (size 1.27 1.27)) (justify left bottom))
+  )
+  (text "NRF Power\n" (at 134.62 59.69 0)
+    (effects (font (size 1.27 1.27)) (justify left bottom))
   )
   (symbol (lib_id "promicro:ProMicro") (at 74.93 82.55 0) (unit 1)
@@
     )
   )
-  (symbol (lib_id "Connector_Generic:Conn_01x06") (at 134.62 120.65 0) (unit 1)
-    (in_bom yes) (on_board yes) (dnp no) (fields_autoplaced)
-    (property "Reference" "J3" (at 137.16 120.65 0)
-      (effects (font (size 1.27 1.27)) (justify left))
-    )
-    (property "Value" "Conn_01x06" (at 137.16 123.19 0)
-      (effects (font (size 1.27 1.27)) (justify left))
-    )
-    (property "Footprint" "" (at 134.62 120.65 0)
-      (effects (font (size 1.27 1.27)) hide)
-    )
-    (property "Datasheet" "~" (at 134.62 120.65 0)
-      (effects (font (size 1.27 1.27)) hide)
-    )
+  (symbol (lib_id "Connector_Generic:Conn_01x06") (at 134.62 119.38 0) (unit 1)
+    (in_bom yes) (on_board yes) (dnp no) (fields_autoplaced)
+    (property "Reference" "J3" (at 137.16 119.38 0)
+      (effects (font (size 1.27 1.27)) (justify left))
+    )
+    (property "Value" "Conn_01x06" (at 137.16 121.92 0)
+      (effects (font (size 1.27 1.27)) (justify left))
+    )
+    (property "Footprint" "" (at 134.62 119.38 0)
+      (effects (font (size 1.27 1.27)) hide)
+    )
+    (property "Datasheet" "~" (at 134.62 119.38 0)
+      (effects (font (size 1.27 1.27)) hide)
+    )
